File: EffectsPaddleBoard/ControllerSheet.kicad_sch (KiCad schematic)
At the start: 21 parts, among them J1 Conn_01x03_Pin, J2 Conn_01x06_Pin, J4 Conn_01x04_Pin, SW1 SW_SPDT, SW2 SW_SPDT, SW3 SW_SPDT, U1 STM32F405RGTx, Y1 16MHz

Commit message: Began with pcb layout
Parts:
- C1, C10, C2, C3, C4, C5, C7, C8, C9: footprint (none) -> Capacitor_SMD:C_0402_1005Metric
- C6: footprint (none) -> Capacitor_SMD:C_1206_3216Metric
- D1: footprint (none) -> LED_SMD:LED_0402_1005Metric
- J1: footprint (none) -> Connector_PinHeader_2.00mm:PinHeader_1x03_P2.00mm_Vertical
- J2: footprint (none) -> Connector_PinHeader_2.00mm:PinHeader_1x06_P2.00mm_Vertical
- J4: footprint (none) -> Connector_PinHeader_2.00mm:PinHeader_1x04_P2.00mm_Vertical
- R1, R2: footprint (none) -> Resistor_SMD:R_0402_1005Metric
- SW1, SW2, SW3: footprint (none) -> Button_Switch_SMD:SW_SPDT_PCM12
- Y1: footprint (none) -> Crystal:Crystal_SMD_3225-4Pin_3.2x2.5mm
Connections:
- no-connect marks 33 -> 31
Changed lines of the file:
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@@
   (no_connect (at 129.54 133.35))
   (no_connect (at 93.98 77.47))
-  (no_connect (at 97.79 79.375))
   (no_connect (at 93.98 105.41))
   (no_connect (at 93.98 120.65))
@@
   (no_connect (at 129.54 97.79))
   (no_connect (at 93.98 115.57))
-  (no_connect (at 99.06 80.645))
   (no_connect (at 129.54 125.73))
   (no_connect (at 93.98 123.19))
@@
     (stroke (width 0) (type default))
   )
-  (wire (pts (xy 235.585 98.425) (xy 239.395 98.425))
+  (wire (pts (xy 233.68 98.425) (xy 239.395 98.425))
     (stroke (width 0) (type default))
   )
@@
     )
   )
-  (global_label "OSC_PH0" (shape input) (at 235.585 98.425 180) (fields_autoplaced)
+  (global_label "OSC_PH0" (shape input) (at 233.68 98.425 180) (fields_autoplaced)
     (effects (font (size 1.27 1.27)) (justify right))
-    (property "Intersheetrefs" "${INTERSHEET_REFS}" (at 224.0916 98.425 0)
+    (property "Intersheetrefs" "${INTERSHEET_REFS}" (at 222.1866 98.425 0)
       (effects (font (size 1.27 1.27)) (justify right) hide)
     )
@@
       (effects (font (size 1.27 1.27)) (justify left))
     )
-    (property "Footprint" "" (at 50.4952 44.45 0)
+    (property "Footprint" "Capacitor_SMD:C_0402_1005Metric" (at 50.4952 44.45 0)
       (effects (font (size 1.27 1.27)) hide)
     )
@@
       (effects (font (size 1.27 1.27)) (justify right))
     )
-    (property "Footprint" "" (at 262.255 43.18 0)
+    (property "Footprint" "Connector_PinHeader_2.00mm:PinHeader_1x06_P2.00mm_Vertical" (at 262.255 43.18 0)
       (effects (font (size 1.27 1.27)) hide)
     )
@@
       (effects (font (size 1.27 1.27)))
     )
-    (property "Footprint" "" (at 89.535 170.307 90)
+    (property "Footprint" "Resistor_SMD:R_0402_1005Metric" (at 89.535 170.307 90)
       (effects (font (size 1.27 1.27)) hide)
     )
@@
       (effects (font (size 1.27 1.27)) (justify left))
     )
-    (property "Footprint" "" (at 39.0652 44.45 0)
+    (property "Footprint" "Capacitor_SMD:C_0402_1005Metric" (at 39.0652 44.45 0)
       (effects (font (size 1.27 1.27)) hide)
     )
@@
       (effects (font (size 1.27 1.27)) (justify left))
     )
-    (property "Footprint" "" (at 35.2552 80.01 0)
+    (property "Footprint" "Capacitor_SMD:C_0402_1005Metric" (at 35.2552 80.01 0)
       (effects (font (size 1.27 1.27)) hide)
     )
@@
       (effects (font (size 1.27 1.27)) (justify right))
     )
-    (property "Footprint" "" (at 101.6 182.245 0)
+    (property "Footprint" "LED_SMD:LED_0402_1005Metric" (at 101.6 182.245 0)
       (effects (font (size 1.27 1.27)) hide)
     )
@@
       (effects (font (size 1.27 1.27)))
     )
-    (property "Footprint" "" (at 25.4 142.24 0)
+    (property "Footprint" "Connector_PinHeader_2.00mm:PinHeader_1x04_P2.00mm_Vertical" (at 25.4 142.24 0)
       (effects (font (size 1.27 1.27)) hide)
     )
@@
       (effects (font (size 1.27 1.27)))
     )
-    (property "Footprint" "" (at 248.92 98.425 0)
+    (property "Footprint" "Crystal:Crystal_SMD_3225-4Pin_3.2x2.5mm" (at 248.92 98.425 0)
       (effects (font (size 1.27 1.27)) hide)
     )
@@
       (effects (font (size 1.27 1.27)) (justify left))
     )
-    (property "Footprint" "" (at 63.1952 44.45 0)
+    (property "Footprint" "Capacitor_SMD:C_0402_1005Metric" (at 63.1952 44.45 0)
       (effects (font (size 1.27 1.27)) hide)
     )
@@
       (effects (font (size 1.27 1.27)) (justify left))
     )
-    (property "Footprint" "" (at 260.0452 111.125 0)
+    (property "Footprint" "Capacitor_SMD:C_0402_1005Metric" (at 260.0452 111.125 0)
       (effects (font (size 1.27 1.27)) hide)
     )
@@
       (effects (font (size 1.27 1.27)))
     )
-    (property "Footprint" "" (at 249.555 147.955 0)
+    (property "Footprint" "Button_Switch_SMD:SW_SPDT_PCM12" (at 249.555 147.955 0)
       (effects (font (size 1.27 1.27)) hide)
     )
@@
       (effects (font (size 1.27 1.27)) (justify left))
     )
-    (property "Footprint" "" (at 74.6252 44.45 0)
+    (property "Footprint" "Capacitor_SMD:C_0402_1005Metric" (at 74.6252 44.45 0)
       (effects (font (size 1.27 1.27)) hide)
     )
@@
       (effects (font (size 1.27 1.27)) (justify left))
     )
-    (property "Footprint" "" (at 240.3602 111.125 0)
+    (property "Footprint" "Capacitor_SMD:C_0402_1005Metric" (at 240.3602 111.125 0)
       (effects (font (size 1.27 1.27)) hide)
     )
@@
       (effects (font (size 1.27 1.27)))
     )
-    (property "Footprint" "" (at 55.88 88.9 0)
+    (property "Footprint" "Button_Switch_SMD:SW_SPDT_PCM12" (at 55.88 88.9 0)
       (effects (font (size 1.27 1.27)) hide)
     )
@@
       (effects (font (size 1.27 1.27)))
     )
-    (property "Footprint" "" (at 85.09 61.468 90)
+    (property "Footprint" "Resistor_SMD:R_0402_1005Metric" (at 85.09 61.468 90)
       (effects (font (size 1.27 1.27)) hide)
     )
@@
       (effects (font (size 1.27 1.27)) (justify left))
     )
-    (property "Footprint" "" (at 27.6352 44.45 0)
+    (property "Footprint" "Capacitor_SMD:C_1206_3216Metric" (at 27.6352 44.45 0)
       (effects (font (size 1.27 1.27)) hide)
     )
@@
       (effects (font (size 1.27 1.27)))
     )
-    (property "Footprint" "" (at 24.765 182.88 0)
+    (property "Footprint" "Connector_PinHeader_2.00mm:PinHeader_1x03_P2.00mm_Vertical" (at 24.765 182.88 0)
       (effects (font (size 1.27 1.27)) hide)
     )
@@
       (effects (font (size 1.27 1.27)))
     )
-    (property "Footprint" "" (at 46.99 68.58 0)
+    (property "Footprint" "Button_Switch_SMD:SW_SPDT_PCM12" (at 46.99 68.58 0)
       (effects (font (size 1.27 1.27)) hide)
     )
@@
       (effects (font (size 1.27 1.27)) (justify left))
     )
-    (property "Footprint" "" (at 35.2552 64.77 0)
+    (property "Footprint" "Capacitor_SMD:C_0402_1005Metric" (at 35.2552 64.77 0)
       (effects (font (size 1.27 1.27)) hide)
     )
@@
       (effects (font (size 1.27 1.27)) (justify left))
     )
-    (property "Footprint" "" (at 86.0552 44.45 0)
-      (effects (font (size 1.27 1.27)) hide)
-    )
+    (property "Footprint" "Capacitor_SMD:C_0402_1005Metric" (at 86.0552 44.45 0)
+      (effects (font (size 1.27 1.27)) hide)
+    )

Commit message: Reviev by David and netnaming
Other:
- note added: "entprellen"
- note added: "von wo kam das?"
Changed lines of the file:
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@@
     (effects (font (size 4 4)) (justify left bottom))
+  )
+  (text "von wo kam das?" (at 23.495 69.215 0)
+    (effects (font (size 1.27 1.27)) (justify left bottom))
   )
   (text "PWR_LED" (at 62.23 165.735 0)
@@
     (effects (font (size 4 4)) (justify left bottom))
   )
+  (text "entprellen" (at 238.125 154.305 0)
+    (effects (font (size 1.27 1.27)) (justify left bottom))
+  )
   (text "JTAG" (at 14.605 125.095 0)

Commit message: Finished layout
Connections:
- net Codec_Reset: now reaches SW2.2 (B), U1.7 (NRST)
Changed lines of the file:
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@@
   (junction (at 239.395 98.425) (diameter 0) (color 0 0 0 0)
+  )
+  (junction (at 66.04 54.61) (diameter 0) (color 0 0 0 0)
   )
   (junction (at 62.23 33.02) (diameter 0) (color 0 0 0 0)
@@
     (stroke (width 0) (type default))
   )
+  (wire (pts (xy 59.055 54.61) (xy 66.04 54.61))
+    (stroke (width 0) (type default))
+  )
   (wire (pts (xy 239.395 113.03) (xy 248.92 113.03))
     (stroke (width 0) (type default))
@@
     )
   )
+  (global_label "Codec_Reset" (shape input) (at 59.055 54.61 180) (fields_autoplaced)
+    (effects (font (size 1.27 1.27)) (justify right))
+    (property "Intersheetrefs" "${INTERSHEET_REFS}" (at 44.2354 54.61 0)
+      (effects (font (size 1.27 1.27)) (justify right) hide)
+    )
+  )
