File: EffectsPaddleBoard/EffectsPaddleBoard.kicad_pcb (KiCad board)
At the start: 4 copper layers, 113.6 x 84.6 mm, 121 parts, among them J1 Conn_01x03_Pin, J2 Conn_01x06_Pin, J3 Barrel_Jack, J4 Conn_01x04_Pin, J5 AudioJack2, J6 AudioJack2, SW1 SW_SPDT, SW2 SW_Push, SW3 SW_SPDT, U1 STM32F405RGTx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

Commit message: Added note for reviewer
Other:
- board text added: "Barreljack, Audiojacks and this potentiometer won't be on the PCB"
- board text removed: "Move the potentiometer so that the adjustment screw is accessible or use a horizontal one."
Changed lines of the file:
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@@
   (gr_line (start 229.8 130.8) (end 125.8 130.8)
     (stroke (width 0.1) (type default)) (layer "Edge.Cuts"))
-  (gr_text "Move the switches to the pcb edge or change them to horizontal ones." (at 116.84 127 90) (layer "Cmts.User")
+  (gr_text "Barreljack, Audiojacks and this\npotentiometer won't be on the PCB" (at 194.2 127.2) (layer "F.SilkS")
     (effects (font (size 1 1) (thickness 0.15)) (justify left bottom))
   )
-  (gr_text "Move the potentiometer so that the adjustment screw\nis accessible or use a horizontal one." (at 182.88 129.54) (layer "Cmts.User")
+  (gr_text "Move the switches to the pcb edge or change them to horizontal ones." (at 116.84 127 90) (layer "Cmts.User")
     (effects (font (size 1 1) (thickness 0.15)) (justify left bottom))
   )
@@
     (effects (font (size 1 1) (thickness 0.15)) (justify left bottom))
   )
-  (gr_text "Would move them as close\nas possible to the codec" (at 180.34 106.68) (layer "Cmts.User")
+  (gr_text "Would move them as close\nas possible to the codec" (at 204.1 100.4) (layer "Cmts.User")
     (effects (font (size 1 1) (thickness 0.15)) (justify left bottom))
   )

Commit message: Corrections, see comments
Parts:
- moved C19 0.87 mm to (173.4, 102.5)
- moved C20 0.87 mm to (176.0, 102.5)
- moved R16 0.87 mm to (171.4, 101.9)
- moved R17 0.87 mm to (178.0, 101.4)
- moved R18 0.87 mm to (170.2, 101.9)
Routing:
- net I2C_SCL: track 3.72 -> 21.5 mm, vias 0 -> 2
- net I2C_SDA: track 3.72 -> 18.3 mm
- net GND: vias 11 -> 13
- added copper zone on B.Cu, net GND
- added copper zone on F.Cu, net GND
Changed lines of the file:
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@@
   )
   (footprint "Resistor_SMD:R_0402_1005Metric" (layer "F.Cu")
-    (at 171 101.115 -90)
+    (at 171.4 101.89 -90)
     (descr "Resistor SMD 0402 (1005 Metric), square (rectangular) end terminal, IPC_7351 nominal, (Body size source: IPC-SM-782 page 72, https://www.pcb-3d.com/wordpress/wp-content/uploads/ipc-sm-782a_amendment_1_and_2.pdf), generated with kicad-footprint-generator")
     (tags "resistor")
@@
   )
   (footprint "Capacitor_SMD:C_1206_3216Metric" (layer "F.Cu")
-    (at 173 101.725 -90)
+    (at 173.4 102.5 -90)
     (descr "Capacitor SMD 1206 (3216 Metric), square (rectangular) end terminal, IPC_7351 nominal, (Body size source: IPC-SM-782 page 76, https://www.pcb-3d.com/wordpress/wp-content/uploads/ipc-sm-782a_amendment_1_and_2.pdf), generated with kicad-footprint-generator")
     (tags "capacitor")
@@
   )
   (footprint "Resistor_SMD:R_0402_1005Metric" (layer "F.Cu")
-    (at 177.6 100.625 -90)
+    (at 178 101.4 -90)
     (descr "Resistor SMD 0402 (1005 Metric), square (rectangular) end terminal, IPC_7351 nominal, (Body size source: IPC-SM-782 page 72, https://www.pcb-3d.com/wordpress/wp-content/uploads/ipc-sm-782a_amendment_1_and_2.pdf), generated with kicad-footprint-generator")
     (tags "resistor")
@@
   )
   (footprint "Resistor_SMD:R_0402_1005Metric" (layer "F.Cu")
-    (at 169.75 101.115 -90)
+    (at 170.15 101.89 -90)
     (descr "Resistor SMD 0402 (1005 Metric), square (rectangular) end terminal, IPC_7351 nominal, (Body size source: IPC-SM-782 page 72, https://www.pcb-3d.com/wordpress/wp-content/uploads/ipc-sm-782a_amendment_1_and_2.pdf), generated with kicad-footprint-generator")
     (tags "resistor")
@@
   )
   (footprint "Capacitor_SMD:C_1206_3216Metric" (layer "F.Cu")
-    (at 175.6 101.725 -90)
+    (at 176 102.5 -90)
     (descr "Capacitor SMD 1206 (3216 Metric), square (rectangular) end terminal, IPC_7351 nominal, (Body size source: IPC-SM-782 page 76, https://www.pcb-3d.com/wordpress/wp-content/uploads/ipc-sm-782a_amendment_1_and_2.pdf), generated with kicad-footprint-generator")
     (tags "capacitor")
@@
   (segment (start 148.675 90.8) (end 148.675 92.055) (width 0.5) (layer "F.Cu") (net 2))
   (segment (start 147.5 94.825) (end 147.5 93.23) (width 0.3) (layer "F.Cu") (net 2))
-  (via (at 172.6 96.6) (size 0.8) (drill 0.4) (layers "F.Cu" "B.Cu") (net 2))
-  (via (at 143.2 94.6) (size 0.8) (drill 0.4) (layers "F.Cu" "B.Cu") (net 2))
-  (via (at 138.6 102.2) (size 0.8) (drill 0.4) (layers "F.Cu" "B.Cu") (net 2))
-  (via (at 174.8 94.4) (size 0.8) (drill 0.4) (layers "F.Cu" "B.Cu") (net 2))
-  (via (at 174.8 96.6) (size 0.8) (drill 0.4) (layers "F.Cu" "B.Cu") (net 2))
-  (via (at 155.6 108.6) (size 0.8) (drill 0.4) (layers "F.Cu" "B.Cu") (net 2))
-  (via (at 140.3 96.3) (size 0.8) (drill 0.4) (layers "F.Cu" "B.Cu") (net 2))
-  (via (at 147.5 96.6) (size 0.8) (drill 0.4) (layers "F.Cu" "B.Cu") (net 2))
-  (via (at 160.2 96.7) (size 0.8) (drill 0.4) (layers "F.Cu" "B.Cu") (net 2))
-  (via (at 172.6 94.4) (size 0.8) (drill 0.4) (layers "F.Cu" "B.Cu") (net 2))
-  (via (at 147.5 104.1) (size 0.8) (drill 0.4) (layers "F.Cu" "B.Cu") (net 2))
+  (via (at 172.6 96.6) (size 0.6) (drill 0.3) (layers "F.Cu" "B.Cu") (net 2))
+  (via (at 163.5 101) (size 0.6) (drill 0.3) (layers "F.Cu" "B.Cu") (free) (net 2))
+  (via (at 143.2 94.6) (size 0.6) (drill 0.3) (layers "F.Cu" "B.Cu") (net 2))
+  (via (at 138.6 102.2) (size 0.6) (drill 0.3) (layers "F.Cu" "B.Cu") (net 2))
+  (via (at 174.8 94.4) (size 0.6) (drill 0.3) (layers "F.Cu" "B.Cu") (net 2))
+  (via (at 162.75 104) (size 0.6) (drill 0.3) (layers "F.Cu" "B.Cu") (free) (net 2))
+  (via (at 174.8 96.6) (size 0.6) (drill 0.3) (layers "F.Cu" "B.Cu") (net 2))
+  (via (at 155.6 108.6) (size 0.6) (drill 0.3) (layers "F.Cu" "B.Cu") (net 2))
+  (via (at 140.3 96.3) (size 0.6) (drill 0.3) (layers "F.Cu" "B.Cu") (net 2))
+  (via (at 147.5 96.6) (size 0.6) (drill 0.3) (layers "F.Cu" "B.Cu") (net 2))
+  (via (at 160.2 96.7) (size 0.6) (drill 0.3) (layers "F.Cu" "B.Cu") (net 2))
+  (via (at 172.6 94.4) (size 0.6) (drill 0.3) (layers "F.Cu" "B.Cu") (net 2))
+  (via (at 147.5 104.1) (size 0.6) (drill 0.3) (layers "F.Cu" "B.Cu") (net 2))
   (segment (start 138.6 98.1) (end 138.6 98) (width 0.3) (layer "F.Cu") (net 5))
   (segment (start 142.25 98.75) (end 142 98.5) (width 0.3) (layer "F.Cu") (net 5))
@@
   (segment (start 145.075 99.25) (end 142.31 99.25) (width 0.3) (layer "F.Cu") (net 6))
   (segment (start 142 99.56) (end 140.94 99.56) (width 0.3) (layer "F.Cu") (net 6))
-  (via (at 187.2 90.6) (size 0.8) (drill 0.4) (layers "F.Cu" "B.Cu") (free) (net 8))
-  (via (at 187.2 92.7) (size 0.8) (drill 0.4) (layers "F.Cu" "B.Cu") (free) (net 8))
+  (via (at 187.2 90.6) (size 0.6) (drill 0.3) (layers "F.Cu" "B.Cu") (free) (net 8))
+  (via (at 187.2 92.7) (size 0.6) (drill 0.3) (layers "F.Cu" "B.Cu") (free) (net 8))
   (segment (start 152 94.825) (end 152 87.75) (width 0.3) (layer "F.Cu") (net 26))
   (segment (start 152.5 89.25) (end 154 87.75) (width 0.3) (layer "F.Cu") (net 27))
@@
   (segment (start 151.5 95.701041) (end 152.248959 96.45) (width 0.3) (layer "F.Cu") (net 35))
   (segment (start 152.248959 96.45) (end 155.25 96.45) (width 0.3) (layer "F.Cu") (net 35))
+  (segment (start 170.5 100) (end 172 100) (width 0.3) (layer "F.Cu") (net 40))
+  (segment (start 161.1595 99.91) (end 162.5 101.2505) (width 0.3) (layer "F.Cu") (net 40))
+  (segment (start 160 99.91) (end 161.1595 99.91) (width 0.3) (layer "F.Cu") (net 40))
+  (segment (start 167.5 103) (end 170.5 100) (width 0.3) (layer "F.Cu") (net 40))
   (segment (start 156.425 100.25) (end 159.66 100.25) (width 0.3) (layer "F.Cu") (net 40))
+  (segment (start 172 100) (end 172.5 99.5) (width 0.3) (layer "F.Cu") (net 40))
+  (segment (start 172.5 99.5) (end 172.5 98) (width 0.3) (layer "F.Cu") (net 40))
+  (segment (start 162.5 103) (end 167.5 103) (width 0.3) (layer "F.Cu") (net 40))
   (segment (start 159.66 100.25) (end 160 99.91) (width 0.3) (layer "F.Cu") (net 40))
+  (via (at 162.5 103) (size 0.6) (drill 0.3) (layers "F.Cu" "B.Cu") (net 40))
+  (via (at 162.5 101.2505) (size 0.6) (drill 0.3) (layers "F.Cu" "B.Cu") (net 40))
+  (segment (start 162.5 101.2505) (end 162.5 103) (width 0.3) (layer "B.Cu") (net 40))
+  (segment (start 161 102) (end 166.5 102) (width 0.3) (layer "F.Cu") (net 41))
+  (segment (start 169 99.5) (end 171.5 99.5) (width 0.3) (layer "F.Cu") (net 41))
+  (segment (start 171.5 99.5) (end 172 99) (width 0.3) (layer "F.Cu") (net 41))
   (segment (start 156.425 100.75) (end 159.66 100.75) (width 0.3) (layer "F.Cu") (net 41))
+  (segment (start 160.09 101.09) (end 161 102) (width 0.3) (layer "F.Cu") (net 41))
+  (segment (start 160 101.09) (end 160.09 101.09) (width 0.3) (layer "F.Cu") (net 41))
+  (segment (start 172 99) (end 172 98) (width 0.3) (layer "F.Cu") (net 41))
   (segment (start 159.66 100.75) (end 160 101.09) (width 0.3) (layer "F.Cu") (net 41))
+  (segment (start 166.5 102) (end 169 99.5) (width 0.3) (layer "F.Cu") (net 41))
   (zone (net 8) (net_name "+1V8") (layer "F.Cu") (hatch edge 0.5)
     (priority 2)
@@
     )
   )
-  (zone (net 2) (net_name "GND") (layer "In1.Cu") (hatch edge 0.5)
-    (connect_pads (clearance 0.5))
+  (zone (net 2) (net_name "GND") (layers "F.Cu" "In1.Cu" "In2.Cu" "B.Cu") (hatch edge 0.5)
+    (connect_pads (clearance 0.3))
     (min_thickness 0.25) (filled_areas_thickness no)
     (fill yes (thermal_gap 0.5) (thermal_bridge_width 0.5))
@@
       )
     )
-  )
-  (zone (net 2) (net_name "GND") (layer "In2.Cu") (hatch edge 0.5)
-    (priority 1)
-    (connect_pads (clearance 0.5))
-    (min_thickness 0.25) (filled_areas_thickness no)
-    (fill yes (thermal_gap 0.5) (thermal_bridge_width 0.5))
-    (polygon
-      (pts
-        (xy 119.75 45)
-        (xy 235.5 45.5)
-        (xy 235.5 133.5)
-        (xy 119.25 133.5)
-      )
-    )

Commit message: Corrected the board, now all parts should be right
Parts:
- removed C31, C32: 1u, Capacitor_SMD:C_1206_3216Metric
- removed C40: 470u, Capacitor_SMD:CP_Elec_8x10.5
- removed C44: 220p, Capacitor_SMD:C_0402_1005Metric
- removed C45: 10n, Capacitor_SMD:C_0402_1005Metric
- removed C46, C48, C49: 100n, Capacitor_SMD:C_0402_1005Metric
- removed C50: 10u, Capacitor_SMD:C_1206_3216Metric
- removed D2: B230, Diode_SMD:D_SMB
- removed FB1: 600, Inductor_SMD:L_0603_1608Metric
- removed L1: 15u, Inductor_SMD:L_0603_1608Metric
- removed R19, R20, R24, R25, R26, R31: 10k, Resistor_SMD:R_0402_1005Metric
- removed R21: 4k7, Resistor_SMD:R_1206_3216Metric
- removed R22: 3k9, Resistor_SMD:R_1206_3216Metric
- removed R27, R30: 3k9, Resistor_SMD:R_0402_1005Metric
- removed R28, R29: 4k7, Resistor_SMD:R_0402_1005Metric
- removed R35: 0, Resistor_SMD:R_0402_1005Metric
- removed R6: 68.1k, Resistor_SMD:R_1206_3216Metric
- removed R7: 10.2k, Resistor_SMD:R_1206_3216Metric
- removed R8: 3.24k, Resistor_SMD:R_1206_3216Metric
- removed R9: 30.9k, Resistor_SMD:R_1206_3216Metric
- removed RV1: 100k, Potentiometer_THT:Potentiometer_Bourns_3005_Horizontal
- removed TP1: TestPoint, Connector_Pin:Pin_D1.3mm_L11.0mm
- removed U6, U7: MCP6401T-xLT, Package_TO_SOT_SMD:SOT-353_SC-70-5
- added U8: TPS7A0518PDBZ, Package_TO_SOT_SMD:SOT-23, F.Cu at (171.1, 76.8)
- C11, C13, C15, C17, C33, C35: value 100u -> 100n; footprint Capacitor_SMD:C_1206_3216Metric -> Capacitor_SMD:C_0402_1005Metric
- C12, C14: value 22m -> 22u; footprint Capacitor_SMD:C_1206_3216Metric -> Capacitor_SMD:C_0805_2012Metric
- C16, C18, C34, C36: value 10m -> 10u; footprint Capacitor_SMD:C_1206_3216Metric -> Capacitor_SMD:C_0805_2012Metric
- C19: value 1m -> 1u; footprint Capacitor_SMD:C_1206_3216Metric -> Capacitor_SMD:C_0805_2012Metric
- C20: value 1m -> 47u; footprint Capacitor_SMD:C_1206_3216Metric -> Capacitor_SMD:C_0805_2012Metric
- C21, C30: value 10u -> 1u; footprint Capacitor_SMD:C_1206_3216Metric -> Capacitor_SMD:C_0805_2012Metric
- C22: value 15n -> 1u; footprint Capacitor_SMD:C_0402_1005Metric -> Capacitor_SMD:C_0805_2012Metric
- C23, C8: value 100n -> 1u; footprint Capacitor_SMD:C_0402_1005Metric -> Capacitor_SMD:C_0805_2012Metric
- C24: value 470u -> 1u; footprint Capacitor_SMD:CP_Elec_8x10.5 -> Capacitor_SMD:C_0805_2012Metric
- C25, C26: value 220p -> 1u; footprint Capacitor_SMD:C_0402_1005Metric -> Capacitor_SMD:C_0805_2012Metric
- C27, C41, C42, C43, C6: footprint Capacitor_SMD:C_1206_3216Metric -> Capacitor_SMD:C_0805_2012Metric
- FB2: value 600 -> 100
- L2: footprint Inductor_SMD:L_0603_1608Metric -> Inductor_SMD:L_0805_2012Metric
- R33: value 10k -> 220
- R5: value 332k -> 0; footprint Resistor_SMD:R_1206_3216Metric -> Resistor_SMD:R_0402_1005Metric
- U2: value TPS54233 -> TPS7A0533PDBZ; footprint Package_SO:SOIC-8_3.9x4.9mm_P1.27mm -> Package_TO_SOT_SMD:SOT-23
- U5: value MCP6401T-xLT -> TPS7A0533PDBZ; footprint Package_TO_SOT_SMD:SOT-353_SC-70-5 -> Package_TO_SOT_SMD:SOT-23
- moved C36 106.5 mm to (175.5, 89.0)
- moved C18 98.4 mm to (169.2, 90.5), turned to 180 degrees
- moved C34 95.3 mm to (179.2, 98.2), turned to -90 degrees
- moved C14 95.0 mm to (179.2, 93.2)
- moved C12 93.9 mm to (183.2, 95.8), turned to -90 degrees
- moved C16 93.8 mm to (166.2, 92.2), turned to 90 degrees
- moved C30 61.3 mm to (188.7, 103.8), turned to 90 degrees
- moved C39 50.8 mm to (150.2, 55.0), turned to 180 degrees
- moved R5 45.2 mm to (190.9, 102.8), turned to 180 degrees
- moved R13 39.0 mm to (159.0, 55.0), turned to 0 degrees
- moved C38 38.9 mm to (153.5, 62.0), turned to 0 degrees
- moved TP3 38.6 mm to (177.0, 51.6)
- moved TP4 38.0 mm to (181.5, 51.5)
- moved J6 35.7 mm to (196.9, 81.8), turned to 90 degrees
- moved C24 32.9 mm to (182.2, 80.0), turned to 0 degrees
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Connections:
- C19 pad 2: Analog_In1 -> Net-(C19-Pad2)
- C20 pad 1: /Codec/Analog_In_R -> /Codec/HPL
- C20 pad 2: Analog_In2 -> /Codec/AudioOutBoard
- C21 pad 1: /Barreljack_in -> GND
- C21 pad 2: GND -> +5V
- C22 pad 1: /SS3v3 -> GND
- C22 pad 2: GND -> +3.3V
- C23 pad 1: /b3v3 -> GND
- C23 pad 2: /ph3v3out -> +5V
- C24 pad 1: +3.3V -> GND
- C24 pad 2: GND -> +3.3VA
- C25 pad 1: /comp3v3 -> GND
- C25 pad 2: GND -> +5V
- C26 pad 1: /comp3v3 -> GND
- C26 pad 2: Net-(C26-Pad2) -> +1V8
- C30 pad 1: +3.3VA -> /Codec/Analog_In_R
- C30 pad 2: GND -> Net-(C30-Pad2)
- J5 pad T: /Analog_FrontBackend/AudioInBoard -> Net-(C19-Pad2)
- J6 pad T: /Analog_FrontBackend/AudioOutBoard -> /Codec/AudioOutBoard
- R23 pad 1: /Analog_FrontBackend/AudioInBoard -> /Codec/Analog_In_R
- R23 pad 2: /Analog_FrontBackend/InLP -> GND
- R5 pad 1: /Barreljack_in -> Net-(C19-Pad2)
- R5 pad 2: /en3v3 -> Net-(C30-Pad2)
- U2 pad 1: /b3v3 -> GND
- U2 pad 2: /Barreljack_in -> +3.3V
- U2 pad 3: /en3v3 -> +5V
- U3 pad 19: Audio_M -> unconnected-(U3-SPKM-Pad19)
- U3 pad 22: Audio_P -> unconnected-(U3-SPKP-Pad22)
- U3 pad 23: Audio_M -> unconnected-(U3-SPKM-Pad19)
- U3 pad 26: Audio_P -> unconnected-(U3-SPKP-Pad22)
- U3 pad 30: /Codec/HPR -> unconnected-(U3-HPR-Pad30)
- U5 pad 1: Analog_In1 -> GND
- U5 pad 2: GND -> +3.3VA
- U5 pad 3: /Analog_FrontBackend/InSigAudio -> +5V
Routing:
- net +1V8: vias 2 -> 0
- removed copper zone on F.Cu, net +1V8
Other:
- board size 113.6 x 84.6 mm -> 91.3 x 77.8 mm
- board text removed: "Barreljack, Audiojacks and this potentiometer won't be on the PCB"
- board text removed: "Would move them as close as possible to the codec"

Commit message: Layout completed
Parts:
- added C31: 47u, Capacitor_SMD:C_0805_2012Metric, F.Cu at (197.4, 77.8)
- added D2: LED, LED_SMD:LED_0402_1005Metric, F.Cu at (173.8, 72.5)
- added R6: 0, Resistor_SMD:R_0402_1005Metric, F.Cu at (197.0, 80.4)
- added R7: 220, Resistor_SMD:R_0402_1005Metric, F.Cu at (173.8, 70.0)
- added RV1: 10k, Potentiometer_THT:Potentiometer_ACP_CA9-H2,5_Horizontal, F.Cu at (177.5, 109.5)
- moved SW2 31.3 mm to (140.1, 79.6), turned to 0 degrees
- moved R33 27.5 mm to (136.1, 84.8), turned to -90 degrees
- moved C8 25.5 mm to (135.6, 87.0), turned to 180 degrees
- moved R23 24.3 mm to (190.3, 82.8), turned to 180 degrees
- moved C30 21.6 mm to (193.6, 82.8), turned to 0 degrees
- moved C41 19.3 mm to (168.2, 66.5), turned to 90 degrees
- moved R5 18.2 mm to (194.6, 85.0), turned to 90 degrees
- moved C19 17.4 mm to (196.6, 84.5), turned to -90 degrees
- moved C42 16.4 mm to (170.5, 66.5), turned to 90 degrees
- moved FID3 12.5 mm to (135.5, 105.5)
- moved FB2 12.3 mm to (173.2, 67.5), turned to 0 degrees
- moved J6 10.9 mm to (195.0, 71.1), turned to 180 degrees
- moved C43 10.3 mm to (176.0, 66.5), turned to 90 degrees
- moved H4 10.1 mm to (205.8, 109.2)
- moved H1 10.0 mm to (125.8, 109.2)
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Connections:
- R18 pad 1: /Codec/Volume -> +3.3VA
- R18 pad 2: GND -> /Codec/VolumeVDiv
- U3 pad 30: unconnected-(U3-HPR-Pad30) -> Net-(U3-HPR)
Routing:
- net GND: track 21.7 -> 32.8 mm, vias 13 -> 14
- net /en5v: track 0.00 -> 6.43 mm
- net /SS5v: track 0.00 -> 1.77 mm
- added copper zone on F.Cu, net /Barreljack_in
Other:
- board size 91.3 x 77.8 mm -> 89.6 x 66.6 mm
- board text removed: "In general, make yourself clear if you want the periapherals connected from the sides or from top."
- board text removed: "Make clear seperatrion between analog and digital parts of your circuit. E.g. now the ferrit pi filter is located on the opposit side of where it is needed."
- board text removed: "Mark clearly which connector does what. You don't want to grill your guitar."
- board text removed: "Move the switches to the pcb edge or change them to horizontal ones."

Commit message: Signal routing almost done
Parts:
- moved R1 21.7 mm to (128.9, 93.7), turned to 0 degrees
- moved R23 20.0 mm to (187.1, 102.6), turned to -90 degrees
- moved C30 17.7 mm to (187.1, 99.3), turned to 90 degrees
- moved R5 14.3 mm to (189.4, 98.3), turned to 180 degrees
- moved C19 14.1 mm to (188.9, 96.3), turned to 0 degrees
- moved R18 10.0 mm to (178.3, 110.5)
- moved R2 7.24 mm to (150.0, 91.2), turned to -90 degrees
- moved RV1 6.28 mm to (183.6, 111.0)
- moved D1 6.08 mm to (149.7, 88.5), turned to -90 degrees
- moved J5 5.37 mm to (195.4, 96.3), turned to 90 degrees
- moved R16 4.94 mm to (178.4, 103.1)
- moved R17 4.91 mm to (180.0, 103.1)
- moved C17 0.67 mm to (169.6, 93.2)
- moved D2 0.59 mm to (174.0, 71.9)
- moved R7 0.59 mm to (174.0, 69.4)
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Routing:
- net Codec_Reset: track 0.00 -> 65.3 mm
- net Net-(U3-HPR): track 0.00 -> 40.0 mm
- net On-Switch: track 0.00 -> 37.2 mm, vias 0 -> 2
- net +1V8: track 0.00 -> 29.1 mm, vias 0 -> 2
- net /fb5v: track 0.00 -> 28.9 mm
- net I2S_ext_SD: track 0.00 -> 28.8 mm, vias 0 -> 2
- net I2S_SD: track 0.00 -> 28.7 mm, vias 0 -> 2
- net I2S_CK: track 0.00 -> 28.2 mm, vias 0 -> 2
- net /Codec/HPL: track 0.00 -> 26.9 mm
- net +3.3V: track 9.60 -> 34.1 mm, vias 0 -> 8
- net Net-(U1-BOOT0): track 0.00 -> 23.0 mm, vias 0 -> 2
- net I2S_WS: track 0.00 -> 21.4 mm, vias 0 -> 2
- net /Codec/Volume: track 0.00 -> 19.8 mm
- net I2S_MCK: track 0.00 -> 19.0 mm, vias 0 -> 2
- net /Codec/Analog_In_R: track 0.00 -> 18.1 mm, vias 0 -> 2
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- added copper zone on F.Cu, net +3.3VA
- added copper zone on F.Cu, net +5V

Commit message: Added filter simulation and last copperfills on front copper (ugly)
Parts:
- removed C41: 10u, Capacitor_SMD:C_0805_2012Metric
- removed C42, C43: 1u, Capacitor_SMD:C_0805_2012Metric
- removed FB2: 100, Inductor_SMD:L_0603_1608Metric
- moved TP2 27.1 mm to (156.9, 53.2)
- moved R7 2.87 mm to (174.1, 72.3), turned to -90 degrees
- moved D2 2.12 mm to (174.1, 69.8), turned to -90 degrees
Routing:
- net Codec_GPIO: track 0.00 -> 31.2 mm, vias 0 -> 2
- net Codec_Reset: track 65.3 -> 67.3 mm
- net +5V: track 13.1 -> 14.8 mm, vias 6 -> 9
- net GND: vias 33 -> 35
- net +3.3VA: vias 4 -> 5
