File: EffectsPaddleBoard/AFB.kicad_sch (KiCad schematic)
At the start: 29 parts, among them J5 AudioJack2, J6 AudioJack2, U5 MCP6401T-xLT, U6 MCP6401T-xLT, U7 MCP6401T-xLT

Commit message: Corrections, see comments
Parts:
- removed C44: 220p, Capacitor_SMD:C_0402_1005Metric, symbol Device:C_Small
- removed C45: 10n, Capacitor_SMD:C_0402_1005Metric, symbol Device:C_Small
- removed C46: 100n, Capacitor_SMD:C_0402_1005Metric, symbol Device:C_Small
- removed C50: 10u, Capacitor_SMD:C_1206_3216Metric, symbol Device:C_Small
- removed J5, J6: AudioJack2, Connector_Audio:Jack_6.35mm_Neutrik_NJ2FD-V_Vertical, symbol Connector_Audio:AudioJack2
- removed R23, R24, R25, R26: 10k, Resistor_SMD:R_0402_1005Metric, symbol Device:R_Small
- removed R35: 0, Resistor_SMD:R_0402_1005Metric, symbol Device:R_Small
- removed U5: MCP6401T-xLT, Package_TO_SOT_SMD:SOT-353_SC-70-5, symbol Amplifier_Operational:MCP6401T-xLT
Other:
- note removed: "DC-decoupling at codec page"
- note removed: "Input Amplitude?"
- note removed: "closely look again...seems sus"

Commit message: Corrected the board, now all parts should be right
Parts:
- removed C48, C49: 100n, Capacitor_SMD:C_0402_1005Metric, symbol Device:C_Small
- removed R27, R30: 3k9, Resistor_SMD:R_0402_1005Metric, symbol Device:R_Small
- removed R28, R29: 4k7, Resistor_SMD:R_0402_1005Metric, symbol Device:R_Small
- removed R31: 10k, Resistor_SMD:R_0402_1005Metric, symbol Device:R_Small
- removed RV1: 100k, Potentiometer_THT:Potentiometer_Bourns_3005_Horizontal, symbol Device:R_Potentiometer
- removed U6, U7: MCP6401T-xLT, Package_TO_SOT_SMD:SOT-353_SC-70-5, symbol Amplifier_Operational:MCP6401T-xLT

Commit message: exported symbols and footprints, updated PCB
Parts:
- FID1, FID2, FID3: symbol Mechanical:Fiducial -> EffectsPaddleBoard:Fiducial
- H1, H2, H3, H4: symbol Mechanical:MountingHole -> EffectsPaddleBoard:MountingHole
Changed lines of the file:
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@@
     (effects (font (size 4 4)) (justify left bottom))
   )
-  (symbol (lib_id "Mechanical:MountingHole") (at 248.92 26.67 0) (unit 1)
+  (symbol (lib_id "EffectsPaddleBoard:MountingHole") (at 248.92 26.67 0) (unit 1)
     (in_bom no) (on_board yes) (dnp no) (fields_autoplaced)
     (property "Reference" "H2" (at 251.46 26.035 0)
@@
     )
   )
-  (symbol (lib_id "Mechanical:MountingHole") (at 226.06 38.735 0) (unit 1)
+  (symbol (lib_id "EffectsPaddleBoard:MountingHole") (at 226.06 38.735 0) (unit 1)
     (in_bom no) (on_board yes) (dnp no) (fields_autoplaced)
     (property "Reference" "H3" (at 228.6 38.1 0)
@@
     )
   )
-  (symbol (lib_id "Mechanical:Fiducial") (at 227.965 53.34 0) (unit 1)
+  (symbol (lib_id "EffectsPaddleBoard:Fiducial") (at 227.965 53.34 0) (unit 1)
     (in_bom no) (on_board yes) (dnp no) (fields_autoplaced)
     (property "Reference" "FID1" (at 231.14 52.705 0)
@@
     )
   )
-  (symbol (lib_id "Mechanical:MountingHole") (at 226.06 26.67 0) (unit 1)
+  (symbol (lib_id "EffectsPaddleBoard:MountingHole") (at 226.06 26.67 0) (unit 1)
     (in_bom no) (on_board yes) (dnp no) (fields_autoplaced)
     (property "Reference" "H1" (at 228.6 26.035 0)
@@
     )
   )
-  (symbol (lib_id "Mechanical:Fiducial") (at 264.16 54.61 0) (unit 1)
+  (symbol (lib_id "EffectsPaddleBoard:Fiducial") (at 264.16 54.61 0) (unit 1)
     (in_bom no) (on_board yes) (dnp no) (fields_autoplaced)
     (property "Reference" "FID3" (at 267.335 53.975 0)
@@
     )
   )
-  (symbol (lib_id "Mechanical:MountingHole") (at 248.92 38.735 0) (unit 1)
+  (symbol (lib_id "EffectsPaddleBoard:MountingHole") (at 248.92 38.735 0) (unit 1)
     (in_bom no) (on_board yes) (dnp no) (fields_autoplaced)
     (property "Reference" "H4" (at 251.46 38.1 0)
@@
     )
   )
-  (symbol (lib_id "Mechanical:Fiducial") (at 246.38 53.975 0) (unit 1)
+  (symbol (lib_id "EffectsPaddleBoard:Fiducial") (at 246.38 53.975 0) (unit 1)
     (in_bom no) (on_board yes) (dnp no) (fields_autoplaced)
     (property "Reference" "FID2" (at 249.555 53.34 0)
